Commit message: add

File: assets/robot.urdf (robot description, URDF)
Before this commit: robot car, 5 links, 4 joints
Links:
- link left_wheel_link: geometry collision cylinder length=0.025 radius=0.06; visual box size=0.10 0.10 0.10

Commit message: add

File: assets/robot.urdf (robot description, URDF)
Before this commit: robot car, 5 links, 4 joints
Links:
- link left_wheel_link: geometry collision cylinder length=0.025 radius=0.06; visual cylinder length=0.025 radius=0.06

Commit message: add

File: assets/robot.urdf (robot description, URDF)
Before this commit: robot car, 5 links, 4 joints
Links:
- link back_caster_link: geometry collision sphere radius=0.014; visual sphere radius=0.015
- link front_caster_link: geometry collision sphere radius=0.014; visual sphere radius=0.015
Joints:
- joint back_caster_joint: type continuous -> fixed
- joint front_caster_joint: type continuous -> fixed
